File: electric/biurko.kicad_sch (KiCad schematic)
At the start: 31 parts, among them J1 12V input screw terminal, J10 lower limit conn, J11 outer control, J2 12V motors screw terminal, J3 12V logic screw terminal, J4 Conn_01x04, J5 V logic conn, J6 motors driver screw terminal, J7 GND logic conn, J8 inner control, J9 upper limit conn, M1 motor, SW1 callibrate, SW2 debug, SW3 upper limit, SW4 lower limit, SW5 up, SW6 down, U1 opt encoder

Commit message: init code + sync
Parts:
- removed 12V-5V: ~, symbol biurko_lib:Step-down_buck
- removed Arduino: ~, symbol biurko_lib:Arduino_nano
- removed J10: lower limit conn, symbol Connector:Screw_Terminal_01x02
- removed J11: outer control, symbol Connector:Screw_Terminal_01x03
- removed J3: 12V logic screw terminal, symbol Connector:Screw_Terminal_01x02
- removed J5: V logic conn, symbol Connector:Screw_Terminal_01x03
- removed J7: GND logic conn, symbol Connector:Screw_Terminal_01x03
- removed J8: inner control, symbol Connector:Screw_Terminal_01x02
- removed J9: upper limit conn, symbol Connector:Screw_Terminal_01x02
- removed SW2: debug, symbol Switch:SW_SPST
- added Arduino_nano2: ~, Module:Arduino_Nano, symbol biurko_lib:Arduino_nano
- added D2: red, LED_THT:LED_D3.0mm, symbol Device:LED
- added D3: yellow, LED_THT:LED_D3.0mm, symbol Device:LED
- added J11: encoder, symbol Connector:Conn_01x03_Pin
- added J12: outer control, symbol Connector:Conn_01x03_Pin
- added J14, J3: lower limit, Connector_PinHeader_2.54mm:PinHeader_1x02_P2.54mm_Vertical, symbol Connector:Conn_01x02_Pin
- added J15, J2: upper limit, Connector_PinHeader_2.54mm:PinHeader_1x02_P2.54mm_Vertical, symbol Connector:Conn_01x02_Pin
- added J16: current_sensor, Connector_PinHeader_2.54mm:PinHeader_1x03_P2.54mm_Vertical, symbol Connector:Conn_01x03_Pin
- added J4: encoder, Connector_PinHeader_2.54mm:PinHeader_1x03_P2.54mm_Vertical, symbol Connector:Conn_01x03_Pin
- added J5: outer control, Connector_PinHeader_2.54mm:PinHeader_1x03_P2.54mm_Vertical, symbol Connector:Conn_01x03_Pin
- added J6: motor control, Connector_PinHeader_2.54mm:PinHeader_1x03_P2.54mm_Vertical, symbol Connector:Conn_01x03_Pin
- added R1, R2: 220R, Resistor_THT:R_Axial_DIN0204_L3.6mm_D1.6mm_P7.62mm_Horizontal, symbol Device:R_Small
- added U1: step-down buck, Package_DIP:DIP-5-6_W7.62mm_Socket, symbol biurko_lib:Step-down_buck
- added U3: current sensor, symbol biurko_lib:ACS712
- C1: footprint (none) -> Capacitor_THT:CP_Radial_D8.0mm_P3.50mm
- C2: renamed from C3; footprint (none) -> Capacitor_THT:CP_Radial_D8.0mm_P3.50mm
- C3: renamed from C2; footprint (none) -> Capacitor_THT:CP_Axial_L10.0mm_D4.5mm_P15.00mm_Horizontal
- C4: footprint (none) -> Capacitor_THT:CP_Axial_L10.0mm_D4.5mm_P15.00mm_Horizontal
- J1: footprint (none) -> TerminalBlock:TerminalBlock_bornier-2_P5.08mm
- J10: renamed from J4; footprint (none) -> Connector_PinHeader_2.54mm:PinHeader_1x04_P2.54mm_Vertical
- J7: renamed from J2; footprint (none) -> TerminalBlock:TerminalBlock_bornier-2_P5.08mm
- L1: footprint (none) -> Inductor_THT:L_Radial_D10.0mm_P5.00mm_Neosid_SD12_style3
- SW1: footprint (none) -> Button_Switch_THT:SW_PUSH_6mm
- renumbered J6 to J13, SW5 to SW3, SW6 to SW4, SW3 to SW5, SW4 to SW6, U1 to U2, motor_driver to motor_driver1
Connections:
- net +12L: now also U1.1 (IN+)
- net +12P: now also U3.5 (I2); no longer C1.1, C3.1, J1.2 (Pin_2), J7.2 (Pin_2), L1.1
- net +5VL: now also U2. (Vcc), Arduino_nano2.27 (5V), D2.2 (A), D3.2 (A), J11.1 (Pin_1), J16.3 (Pin_3), J4.1 (Pin_1), U3.1 (VCC)
- net GND: now also J10.4 (Pin_4), SW1.1, SW3.1, SW4.1, SW5.1, SW6.1, U2. (Vcc), motor_driver1.4 (GND), Arduino_nano2.29 (GND), Arduino_nano2.4 (GND), J11.3 (Pin_3), J12.3 (Pin_3), J14.2 (Pin_2), J15.2 (Pin_2), J16.1 (Pin_1), J2.2 (Pin_2), J3.2 (Pin_2), J4.3 (Pin_3), J5.3 (Pin_3), J6.3 (Pin_3), U1.3 (OUT-), U3.3 (GND); no longer C2.2, C4.2, NT1.1
- net GND2: now also C2.2, C4.2, NT1.1, U1.2 (IN-); no longer J10.4 (Pin_4), SW1.1, SW3.1, SW4.1, SW5.1, SW6.1, motor_driver1.4 (GND)
- net up: now reaches SW3.2
- net up: now also Arduino_nano2.6 (D3/INT1), J12.1 (Pin_1), J5.1 (Pin_1)
- net down: now reaches SW4.2
- net down: now also Arduino_nano2.7 (D4), J12.2 (Pin_2), J5.2 (Pin_2)
- net upper_lmt: now reaches SW5.2
- net upper_lmt: now also Arduino_nano2.12 (D9), J14.1 (Pin_1), J2.1 (Pin_1)
- net encoder_out: now reaches U2. (Vcc)
- net encoder_out: now also Arduino_nano2.5 (D2/INT0), J11.2 (Pin_2), J4.2 (Pin_2)
- net callibrate_trg: now reaches SW1.2
- net callibrate_trg: now also Arduino_nano2.11 (D8)
- net lower_lmt: now reaches SW6.2
- net lower_lmt: now also Arduino_nano2.13 (D10), J15.1 (Pin_1), J3.1 (Pin_1)
- net DIR renamed dir
- net dir: now also Arduino_nano2.15 (D12/MISO), J6.1 (Pin_1)
- net PWM renamed pwm
- net pwm: now also Arduino_nano2.14 (D11/MOSI), J6.2 (Pin_2)
- new net: D3.1 (K), R2.1
- new net: D2.1 (K), R1.1
- new net +12V: C1.1, C3.1, J1.2 (Pin_2), J7.2 (Pin_2), L1.1, U3.4 (I1)
- new net +7.5V: Arduino_nano2.30 (VIN), U1.4 (OUT+)
- new net error: Arduino_nano2.9 (D6), R1.2
- new net mot_current: Arduino_nano2.19 (A0), J16.2 (Pin_2), U3.2 (OUT)
- new net status: Arduino_nano2.8 (D5), R2.2
- no-connect marks 3 -> 17
Other:
- title: (none) -> Automatic desk v1
- moved on the sheet: C1, C2, C3, C4, C5, C6, C7, J1, J10, J13, J7, L1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
